File: ELS-ELH/ELH/PCB_A/PCB_A.kicad_sch (KiCad schematic)
At the start: 44 parts, among them J1 Conn_01x08_Pin, J3 Conn_01x20_Pin, J4 Conn_01x20_Pin, Q1 IRLZ44N, Q2 IRLZ44N, Q4 IRLZ44N, Q6 IRLZ44N

Commit message: PCB B connection advances
Connections:
- net GND: now also J3.20 (Pin_20); no longer J3.1 (Pin_1)
- net UART1_RX_1: now also J3.14 (Pin_14), J3.15 (Pin_15), J3.16 (Pin_16); no longer J3.5 (Pin_5), J3.6 (Pin_6), J3.7 (Pin_7)
- net UART1_TX_1: now also J3.17 (Pin_17), J3.18 (Pin_18), J3.19 (Pin_19); no longer J3.2 (Pin_2), J3.3 (Pin_3), J3.4 (Pin_4)
Other:
- moved on the sheet: J1
Changed lines of the file:
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@@
 	)
 	(label "VCC"
-		(at 154.94 173.99 180)
+		(at 180.34 58.42 180)
 		(effects
 			(font
@@
 	)
 	(label "UART1_RX_1"
-		(at 137.16 129.54 0)
+		(at 137.16 149.86 0)
 		(effects
 			(font
@@
 		)
 	)
-	(label "UART1_TX_1"
-		(at 137.16 119.38 0)
-		(effects
-			(font
-				(size 1.27 1.27)
-			)
-			(justify left bottom)
-		)
-	)
 	(label "Ch_D_mosfet_1"
 		(at 165.1 157.48 0)
@@
 		)
 	)
+	(label "UART1_RX_1"
+		(at 137.16 147.32 0)
+		(effects
+			(font
+				(size 1.27 1.27)
+			)
+			(justify left bottom)
+		)
+	)
 	(label "BIN2"
 		(at 26.67 163.83 180)
@@
 		)
 	)
-	(label "UART1_RX_1"
-		(at 137.16 127 0)
-		(effects
-			(font
-				(size 1.27 1.27)
-			)
-			(justify left bottom)
-		)
-	)
 	(label "Ch_C_mosfet_1"
 		(at 26.67 118.11 180)
@@
 	)
 	(label "L_IS"
-		(at 133.35 181.61 0)
+		(at 165.1 59.69 0)
 		(effects
 			(font
@@
 		)
 	)
-	(label "UART1_TX_1"
-		(at 137.16 116.84 0)
-		(effects
-			(font
-				(size 1.27 1.27)
-			)
-			(justify left bottom)
-		)
-	)
 	(label "R_IS"
-		(at 133.35 179.07 0)
+		(at 165.1 57.15 0)
 		(effects
 			(font
@@
 	)
 	(label "L_EN"
-		(at 133.35 186.69 0)
+		(at 165.1 64.77 0)
 		(effects
 			(font
@@
 	)
 	(label "VCC"
-		(at 133.35 173.99 0)
+		(at 165.1 52.07 0)
 		(effects
 			(font
@@
 	)
 	(label "UART1_TX_1"
-		(at 137.16 121.92 0)
+		(at 137.16 154.94 0)
 		(effects
 			(font
@@
 	)
 	(label "RPWM"
-		(at 133.35 189.23 0)
+		(at 165.1 67.31 0)
 		(effects
 			(font
@@
 		)
 	)
+	(label "UART1_TX_1"
+		(at 137.16 157.48 0)
+		(effects
+			(font
+				(size 1.27 1.27)
+			)
+			(justify left bottom)
+		)
+	)
 	(label "PWMB"
 		(at 248.92 82.55 0)
@@
 		)
 	)
-	(label "UART1_RX_1"
-		(at 137.16 124.46 0)
+	(label "UART1_TX_1"
+		(at 137.16 160.02 0)
 		(effects
 			(font
@@
 	)
 	(label "GND"
-		(at 133.35 176.53 0)
+		(at 165.1 54.61 0)
 		(effects
 			(font
@@
 	)
 	(label "LPWM"
-		(at 133.35 191.77 0)
+		(at 165.1 69.85 0)
+		(effects
+			(font
+				(size 1.27 1.27)
+			)
+			(justify left bottom)
+		)
+	)
+	(label "UART1_RX_1"
+		(at 137.16 152.4 0)
 		(effects
 			(font
@@
 	)
 	(label "R_EN"
-		(at 133.35 184.15 0)
+		(at 165.1 62.23 0)
 		(effects
 			(font
@@
 	(symbol
 		(lib_id "power:+5V")
-		(at 154.94 173.99 270)
+		(at 180.34 58.42 270)
 		(unit 1)
 		(exclude_from_sim no)
@@
 		(dnp no)
 		(property "Reference" "#PWR022"
-			(at 151.13 173.99 0)
+			(at 176.53 58.42 0)
 			(effects
 				(font
@@
 		)
 		(property "Value" "+5V"
-			(at 157.48 173.99 90)
+			(at 182.88 58.42 90)
 			(effects
 				(font
@@
 		)
 		(property "Footprint" ""
-			(at 154.94 173.99 0)
+			(at 180.34 58.42 0)
 			(effects
 				(font
@@
 		)
 		(property "Datasheet" ""
-			(at 154.94 173.99 0)
+			(at 180.34 58.42 0)
 			(effects
 				(font
@@
 		)
 		(property "Description" "Power symbol creates a global label with name \"+5V\""
-			(at 154.94 173.99 0)
+			(at 180.34 58.42 0)
 			(effects
 				(font
@@
 	(symbol
 		(lib_id "Connector:Conn_01x08_Pin")
-		(at 128.27 181.61 0)
+		(at 160.02 59.69 0)
 		(unit 1)
 		(exclude_from_sim no)
@@
 		(fields_autoplaced yes)
 		(property "Reference" "J1"
-			(at 128.905 168.91 0)
+			(at 160.655 46.99 0)
 			(effects
 				(font
@@
 		)
 		(property "Value" "Conn_01x08_Pin"
-			(at 128.905 171.45 0)
+			(at 160.655 49.53 0)
 			(effects
 				(font
@@
 		)
 		(property "Footprint" "Connector_PinSocket_2.54mm:PinSocket_1x08_P2.54mm_Vertical"
-			(at 128.27 181.61 0)
+			(at 160.02 59.69 0)
 			(effects
 				(font
@@
 		)
 		(property "Datasheet" "~"
-			(at 128.27 181.61 0)
+			(at 160.02 59.69 0)
 			(effects
 				(font
@@
 		)
 		(property "Description" "Generic connector, single row, 01x08, script generated"
-			(at 128.27 181.61 0)
+			(at 160.02 59.69 0)
 			(effects
 				(font
@@
 	(symbol
 		(lib_id "power:GND")
-		(at 137.16 114.3 90)
+		(at 137.16 162.56 90)
 		(unit 1)
 		(exclude_from_sim no)
@@
 		(fields_autoplaced yes)
 		(property "Reference" "#PWR042"
-			(at 143.51 114.3 0)
+			(at 143.51 162.56 0)
 			(effects
 				(font
@@
 		)
 		(property "Value" "GND"
-			(at 140.97 114.2999 90)
+			(at 140.97 162.5599 90)
 			(effects
 				(font
@@
 		)
 		(property "Footprint" ""
-			(at 137.16 114.3 0)
+			(at 137.16 162.56 0)
 			(effects
 				(font
@@
 		)
 		(property "Datasheet" ""
-			(at 137.16 114.3 0)
+			(at 137.16 162.56 0)
 			(effects
 				(font
@@
 		)
 		(property "Description" "Power symbol creates a global label with name \"GND\" , ground"
-			(at 137.16 114.3 0)
+			(at 137.16 162.56 0)
 			(effects
 				(font

Commit message: final updates
Connections:
- net +3V3: now also J1.1 (Pin_1), J3.5 (Pin_5), J3.6 (Pin_6), J3.7 (Pin_7), J4.11 (Pin_11), J4.12 (Pin_12); no longer Driver_DC2.2 (VCC), Teensy3.3.3V_1 (3.3V), Teensy3.3.3V_2 (3.3V), Teensy3.3.3V_3 (3.3V)
- net +5V: now also J3.10 (Pin_10), J3.8 (Pin_8), J3.9 (Pin_9), J4.5 (Pin_5), J4.6 (Pin_6), J4.7 (Pin_7); no longer BOOST1.3 (OUT+), C1.2, C3.1, J1.1 (Pin_1), J4.14 (Pin_14), Teensy3.VIN
- net Ch_C_mosfet_1: now also J4.10 (Pin_10); no longer J4.7 (Pin_7)
- net GND: now also J3.14 (Pin_14), J3.15 (Pin_15), J3.16 (Pin_16), J4.17 (Pin_17), J4.2 (Pin_2), J4.3 (Pin_3), J4.4 (Pin_4)
- net L_EN: now also Teensy3.40 (A16)
- net L_IS: now also Teensy3.38 (A14)
- net R_EN: now also Teensy3.39 (A15)
- net R_IS: now also Teensy3.37 (CS3)
- net UART1_RX_1: now also J3.11 (Pin_11), J3.12 (Pin_12), J3.13 (Pin_13); no longer J3.14 (Pin_14), J3.15 (Pin_15), J3.16 (Pin_16)
- net +5VA: now reaches J3.2 (Pin_2)
- net +5VA: now also BOOST1.3 (OUT+), C1.2, C3.1, J3.3 (Pin_3), J3.4 (Pin_4), J4.14 (Pin_14), J4.15 (Pin_15), J4.16 (Pin_16), Teensy3.VIN
- new net +3.3V: Driver_DC2.2 (VCC), Teensy3.3.3V_1 (3.3V), Teensy3.3.3V_2 (3.3V), Teensy3.3.3V_3 (3.3V)
- no-connect marks 39 -> 35

Commit message: Update on net labels of both PCBs
Parts:
- J3, J4: footprint Connector_PinSocket_2.54mm:PinSocket_1x20_P2.54mm_Vertical -> Connector_PinHeader_2.54mm:PinHeader_1x20_P2.54mm_Vertical
Connections:
- net +12V: no longer Bornera4.2 (Pin_2), Bornera5.2 (Pin_2), C10.1, C9.1, D1.1 (K), D9.1 (K), Regulator3.2 (IN+), Regulator4.4 (OUTPUT+)
- net +5V: now also J3.5 (Pin_5), J3.6 (Pin_6), J3.7 (Pin_7), J4.1 (Pin_1), J4.2 (Pin_2), J4.3 (Pin_3); no longer C2.1, J3.10 (Pin_10), J3.8 (Pin_8), J3.9 (Pin_9), J4.5 (Pin_5), J4.6 (Pin_6), J4.7 (Pin_7), Regulator1.3 (Input), Regulator3.4 (OUTPUT+)
- net +5VA: no longer BOOST1.3 (OUT+), J3.2 (Pin_2), J3.3 (Pin_3), J3.4 (Pin_4), J4.14 (Pin_14), J4.15 (Pin_15), J4.16 (Pin_16)
- net BUZZER2: no longer R9.1
- net Ch_D_mosfet_2: no longer R16.1
- net GND: now also J3.12 (Pin_12), J3.4 (Pin_4), J3.8 (Pin_8), J4.12 (Pin_12), J4.16 (Pin_16), J4.20 (Pin_20), J4.8 (Pin_8); no longer J3.14 (Pin_14), J3.15 (Pin_15), J4.17 (Pin_17), J4.2 (Pin_2), J4.3 (Pin_3)
- net LED4: no longer R8.2
- net LED5: no longer R2.2
- net LED6: no longer R1.2
- net TX_UART_BUS1_3V3: now reaches Teensy3.7 (RX2)
- net TX_UART_BUS1_3V3: now also J3.17 (Pin_17), J3.18 (Pin_18), J3.19 (Pin_19)
- net RX_UART_BUS1_3V3: now reaches Teensy3.8 (TX2)
- net RX_UART_BUS1_3V3: now also J3.13 (Pin_13), J3.14 (Pin_14), J3.15 (Pin_15)
- net +5V_MCU: now reaches J3.1 (Pin_1)
- net +5V_MCU: now also BOOST1.3 (OUT+), C2.1, J3.2 (Pin_2), J3.3 (Pin_3), J4.5 (Pin_5), J4.6 (Pin_6), J4.7 (Pin_7), Regulator1.3 (Input)
- removed net +3V3: C4.1, J1.1 (Pin_1), J3.5 (Pin_5), J3.6 (Pin_6), J3.7 (Pin_7), J4.11 (Pin_11), J4.12 (Pin_12), J4.13 (Pin_13), Regulator1.2 (Output)
- net Ch_C_mosfet_1 renamed +3.3V_SENSORS
- net +3.3V_SENSORS: now also C4.1, J1.1 (Pin_1), J3.10 (Pin_10), J3.11 (Pin_11), J3.9 (Pin_9), J4.11 (Pin_11), Regulator1.2 (Output); no longer J4.8 (Pin_8), R3.1
- net Ch_C_mosfet_2 renamed CH_C_MOSFET_TEENSY_3V3
- net Ch_D_mosfet_1 renamed CH_C_MOSFET_ESP_3V3
- net CH_C_MOSFET_ESP_3V3: now also J4.17 (Pin_17), R3.1; no longer J4.20 (Pin_20), R20.1
- removed net UART1_RX_1: J3.11 (Pin_11), J3.12 (Pin_12), J3.13 (Pin_13), Teensy3.4 (BCLK2)
- removed net UART1_TX_1: J3.17 (Pin_17), J3.18 (Pin_18), J3.19 (Pin_19), Teensy3.0 (RX1)
- new net ACTUATOR_POWER_REG_1: Bornera4.2 (Pin_2), Bornera5.2 (Pin_2), C10.1, C9.1, D1.1 (K), D9.1 (K), Regulator3.2 (IN+), Regulator4.4 (OUTPUT+)
- new net ACTUATOR_POWER_REG_2: Regulator3.4 (OUTPUT+)
- new net BUZZER_SIGNAL_3V3: R9.1
- new net CH_D_MOSFET_ESP_3V3: J4.13 (Pin_13), J4.14 (Pin_14), J4.15 (Pin_15), R20.1
- new net CH_D_MOSFET_TEENSY_3V3: R16.1
- new net LED_BLUE_SIGNAL_3V3: R1.2
- new net LED_GREEN_SIGNAL_3V3: R2.2
- new net LED_RED_SIGNAL_3V3: R8.2
- no-connect marks 35 -> 34
Other:
- moved on the sheet: Q1, Q4, R10, R11, R16, R18, R19, R20, R3, R6
