File: ELS-ELH/ELH/PCB_A/PCB_A.kicad_pcb (KiCad board)
At the start: 2 copper layers, 95 x 95 mm, 82 parts, among them J1 Conn_01x08_Pin, J3 Conn_01x20_Pin, J4 Conn_01x20_Pin, Q1 IRLZ44N, Q2 IRLZ44N, Q3 IRLZ44N, Q4 IRLZ44N, Q5 IRLZ44N, Q6 IRLZ44N

Commit message: PCB B Almost finishhed
Parts:
- removed the BOOST1 at (161.6, -6.13)
- removed the BOOST1 at (-37.4, 20.9)
- removed the BOOST2 at (161.6, 16.4)
- removed the BOOST2 at (0.46, 20.9)
- removed BZ2 (x2): Buzzer, Buzzer_Beeper:Buzzer_12x9.5RM7.6
- removed Bornera1: Camera Connection, ELH_Library:Bornera 2P
- removed Bornera2: Ch.A Output, ELH_Library:Bornera 2P
- removed Bornera3: PWR 3, ELH_Library:Bornera 2P
- removed Bornera4: Ch.C Output, ELH_Library:Bornera 2P
- removed Bornera5: Ch.D Output, ELH_Library:Bornera 2P
- removed Bornera6: Sensor Power Supply, ELH_Library:Bornera 2P
- removed Bornera7: Ch.B Output, ELH_Library:Bornera 2P
- removed Bornera8: Camera Power Supply, ELH_Library:Bornera 2P
- removed C1 (x2), C5: 100nF, Capacitor_THT:C_Disc_D5.0mm_W2.5mm_P5.00mm
- removed the C10 at (29.5, 4.45)
- removed C2: 10uF, Capacitor_THT:CP_Radial_D5.0mm_P2.00mm
- removed C3 (x2): 10uF, Capacitor_THT:CP_Radial_D5.0mm_P2.50mm
- removed the C4 at (21.0, 15.3)
- removed the C6 at (176.0, 48.3)
- removed the C9 at (-14.8, 7.20)
- removed D1, D9: 1N4007, Diode_THT:D_DO-41_SOD81_P10.16mm_Horizontal
- removed the D3 at (195.7, 47.5)
- removed the D3 at (-38.5, -33.3)
- removed Driver_DC2: TB6612FNG, ELH_Library:TB6612FNG
- removed ESP1: ESP32 DEVKIT V1, ELH_Library:ESP32 DEVKIT V1
- removed the J1 at (-8.94, 9.70)
- removed the J1 at (143.4, 25.3)
- removed the J4 at (24.1, 44.0)
- removed R1 (x2), R2 (x2): 330, Resistor_THT:R_Axial_DIN0207_L6.3mm_D2.5mm_P7.62mm_Horizontal
- removed R19, R22, R24: 10K, Resistor_THT:R_Axial_DIN0207_L6.3mm_D2.5mm_P7.62mm_Horizontal
- removed R20, R21, R23, R3, R6: 220, Resistor_THT:R_Axial_DIN0207_L6.3mm_D2.5mm_P7.62mm_Horizontal
- removed the R8 at (131.9, 33.2)
- removed the R8 at (-26.1, -32.8)
- removed the R9 at (131.9, 37.2)
- removed the R9 at (30.9, -7.96)
- removed the Regulator3 at (161.6, -28.7)
- removed the Regulator3 at (31.9, 24.3)
- removed Regulator4: LM2596, ELH_Library:LM2596
- removed Teensy3: Teensy 4.1, ELH_Library:Teensy 4.1
- added BOOST1: TAR-MT3608, ELH_Library:TAR-MT3608, F.Cu at (12.0, 40.9)
- added BOOST2: TAR-MT3608, ELH_Library:TAR-MT3608, F.Cu at (12.0, -22.5)
- added C7: C_Polarized_Small, Capacitor_THT:CP_Radial_D6.3mm_P2.50mm, F.Cu at (28.4, -19.4)
- added C8: C_Polarized_Small, Capacitor_THT:CP_Radial_D6.3mm_P2.50mm, F.Cu at (19.7, -4.30)
- added D2: 1N4007, Diode_THT:D_DO-41_SOD81_P10.16mm_Horizontal, F.Cu at (136.1, 136.4)
- added D3: 1N4007, Diode_THT:D_DO-41_SOD81_P10.16mm_Horizontal, F.Cu at (136.1, 132.1)
- added J10: Screw_Terminal_01x02, ELH_Library:Bornera 2P, F.Cu at (34.4, -0.32)
- added J9: Screw_Terminal_01x02, ELH_Library:Bornera 2P, F.Cu at (34.3, -16.3)
- added R14: R_US, Resistor_THT:R_Axial_DIN0207_L6.3mm_D2.5mm_P7.62mm_Horizontal, F.Cu at (-7.36, -12.2)
- added R15: R_US, Resistor_THT:R_Axial_DIN0207_L6.3mm_D2.5mm_P7.62mm_Horizontal, B.Cu at (-11.6, 15.1)
- added R17: R_US, Resistor_THT:R_Axial_DIN0207_L6.3mm_D2.5mm_P7.62mm_Horizontal, B.Cu at (0.56, 15.1)
- added R7: R_US, Resistor_THT:R_Axial_DIN0207_L6.3mm_D2.5mm_P7.62mm_Horizontal, F.Cu at (-4.06, -12.4)
- added R8: R_US, Resistor_THT:R_Axial_DIN0207_L6.3mm_D2.5mm_P7.62mm_Horizontal, F.Cu at (-4.06, -8.39)
- added R9: R_US, Resistor_THT:R_Axial_DIN0207_L6.3mm_D2.5mm_P7.62mm_Horizontal, B.Cu at (-19.7, 15.1)
- added Regulator2: MP1584, ELH_Library:LM2596, F.Cu at (-28.3, 1.13)
- C10: renamed from C11; value 47uF -> C_Polarized_Small
- C4: renamed from C2; value 10uF -> C_Polarized_Small
- C6: renamed from C7; value 10uF -> C_Polarized_Small
- C9: renamed from C12; value 47uF -> C_Polarized_Small
- J1: renamed from Bornera6; value PWR 1 -> Screw_Terminal_01x02
- J11: renamed from Bornera11; value Ch.A Output -> Screw_Terminal_01x02
- J12: renamed from Bornera10; value Ch. B Output -> Screw_Terminal_01x02
- J2: renamed from Bornera8; value PWR 2 -> Screw_Terminal_01x02
- J3: value Conn_01x20_Pin -> Screw_Terminal_01x02; footprint Connector_PinSocket_2.54mm:PinSocket_1x20_P2.54mm_Vertical -> ELH_Library:Bornera 2P; moved to F.Cu
- J4: renamed from Bornera9; value PWR 4 -> Screw_Terminal_01x02
- J5: renamed from Bornera1; value PWR 2 REG -> Screw_Terminal_01x02
- R10, R11, R18: value 10K -> R_US
- R12: value ~ -> R_US; moved to B.Cu
- R13: value ~ -> R_US
- R16: value 220 -> R_US
- Regulator1: value LM1117T -> MP1584; footprint ELH_Library:LM1117T -> ELH_Library:LM2596
- moved J8 167.9 mm to (-24.1, 44.0), turned to 90 degrees
- moved Q5 159.4 mm to (29.2, 24.6), turned to 90 degrees
- moved Q3 155.3 mm to (31.2, 33.0), turned to 180 degrees
- moved R13 149.2 mm to (-7.36, -8.17), turned to 180 degrees
- moved J1 148.8 mm to (-33.6, 18.9), turned to -90 degrees
- moved J6 148.5 mm to (-24.1, -44.0), turned to 90 degrees
- moved J4 145.2 mm to (-34.1, -15.7), turned to -90 degrees
- moved J2 145.1 mm to (-33.8, 7.29), turned to -90 degrees
- moved J5 144.4 mm to (-34.2, -27.6), turned to -90 degrees
- moved C9 137.4 mm to (19.7, 11.4)
- moved C10 134.9 mm to (20.3, 22.4)
- moved R12 130.0 mm to (4.61, 15.1), turned to 90 degrees
- moved Regulator3 107.4 mm to (89.2, 1.35)
- moved C4 93.2 mm to (240.4, 38.5)
- moved J11 76.2 mm to (34.6, 27.9), turned to 90 degrees
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- renumbered D2 to D5, J3 to J6, J4 to J8, Regulator1 to Regulator3
Connections:
- C10 pad 2: Net-(Bornera10-Pin_1) -> Net-(D5-A)
- C9 pad 2: Net-(Bornera11-Pin_1) -> Net-(D4-A)
- D4 pad 2: Net-(Bornera11-Pin_1) -> Net-(D4-A)
- D5 pad 2: Net-(Bornera10-Pin_1) -> Net-(D5-A)
- J11 pad 1: Net-(Bornera11-Pin_1) -> Net-(D4-A)
- J12 pad 1: Net-(Bornera10-Pin_1) -> Net-(D5-A)
- J3 pad 1: unconnected-(J3-Pin_1-Pad1) -> Net-(J3-Pin_1)
- J3 pad 2: +5VA -> GND
- Q1 pad 2: Net-(Bornera4-Pin_1) -> Net-(D5-A)
- Q1 pad 3: Net-(Q1-S) -> GND
- Q2 pad 2: Net-(Q2-D) -> Net-(D4-A)
- Q3 pad 2: Net-(Bornera10-Pin_1) -> Net-(D2-A)
- Q3 pad 3: GND -> Net-(Q3-S)
- Q4 pad 2: Net-(Q1-S) -> Net-(Q3-S)
- Q5 pad 2: Net-(Bornera11-Pin_1) -> Net-(D3-A)
- Q5 pad 3: GND -> Net-(Q5-S)
- Q6 pad 2: Net-(Bornera5-Pin_1) -> Net-(Q5-S)
- Q6 pad 3: Net-(Q2-D) -> GND
- R10 pad 1: Net-(Q1-G) -> /CH_C_MOSFET_ESP_3V3
- R10 pad 2: GND -> Net-(Q6-G)
- R11 pad 1: Net-(Q4-G) -> /CH_D_MOSFET_ESP2_3V3
- R11 pad 2: GND -> Net-(Q3-G)
- R12 pad 1: /R_IS_BTS7960_3V3 -> /CH_C_MOSFET_ESP2_3V3
- R12 pad 2: Net-(C5-Pad1) -> Net-(Q5-G)
- R13 pad 1: /L_IS_BTS7960_3V3 -> Net-(Q1-G)
- R13 pad 2: Net-(C6-Pad2) -> GND
- R16 pad 1: /CH_D_MOSFET_ESP2_3V3 -> Net-(Q4-G)
- R16 pad 2: Net-(Q6-G) -> GND
Routing:
- net +5V: track 305.9 -> 0.00 mm
- net +12V: track 266.1 -> 0.00 mm
- net +3V3: track 218.6 -> 0.00 mm
- net +5VA: track 213.5 -> 0.00 mm
- net +3.3V: track 71.8 -> 0.00 mm
- net /Ch_C_mosfet_2: track 69.2 -> 0.00 mm
- net Net-(BOOST1-IN+): track 68.1 -> 0.00 mm
- net /Ch_D_mosfet_2: track 64.8 -> 0.00 mm
- net Net-(BOOST2-OUT+): track 58.6 -> 0.00 mm
- net Net-(Bornera7-Pin_2): track 56.4 -> 0.00 mm
- net Net-(Bornera7-Pin_1): track 53.0 -> 0.00 mm
- net /BUZZER2: track 48.8 -> 0.00 mm
- net Net-(Bornera5-Pin_1): track 48.7 -> 0.00 mm
- net Net-(Bornera2-Pin_1): track 44.7 -> 0.00 mm
- net Net-(BOOST2-IN+): track 43.5 -> 0.00 mm
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Other:
- board text removed: "B01"
- board text removed: "BIN1"

Commit message: PCB B ready, PCB A layout ready
Parts:
- removed J8: Conn_01x20_Pin, Connector_PinHeader_2.54mm:PinHeader_1x20_P2.54mm_Vertical
- added J7: Conn_01x20_Pin, Connector_PinHeader_2.54mm:PinHeader_1x20_P2.54mm_Vertical, B.Cu at (-24.1, -44.0)
- D2, D3, D4, D5, J6, R13, R7: moved to B.Cu
- J1: value Screw_Terminal_01x02 -> PWR 1
- J10: value Screw_Terminal_01x02 -> CH C OUT
- J11: value Screw_Terminal_01x02 -> CH A OUT
- J12: value Screw_Terminal_01x02 -> CH B OUT
- J2: value Screw_Terminal_01x02 -> PWR 2
- J3: value Screw_Terminal_01x02 -> PWR 3
- J4: value Screw_Terminal_01x02 -> PWR 4
- J5: value Screw_Terminal_01x02 -> PWR 2 OUT
- J9: value Screw_Terminal_01x02 -> CH D OUT
- moved C4 224.5 mm to (16.2, 28.9)
- moved D3 177.5 mm to (32.2, -11.8), turned to -90 degrees
- moved D2 169.6 mm to (32.1, 2.42), turned to -90 degrees
- moved D4 135.7 mm to (32.2, -26.6), turned to -90 degrees
- moved C6 126.6 mm to (21.9, 28.7)
- moved D5 113.7 mm to (31.2, 26.9), turned to 90 degrees
- moved J6 88.0 mm to (-24.1, 44.0), turned to -90 degrees
- moved Regulator3 78.8 mm to (18.7, 36.6), turned to 180 degrees
- moved R7 44.2 mm to (2.53, 31.2), turned to 180 degrees
- moved J11 41.9 mm to (35.8, -13.9)
- moved Q4 40.7 mm to (18.5, 10.6), turned to 0 degrees
- moved R8 39.0 mm to (28.6, -29.6), turned to 180 degrees
- moved R13 38.0 mm to (-11.2, 29.6)
- moved Q5 35.5 mm to (18.1, -9.18), turned to 0 degrees
- moved C9 34.5 mm to (31.8, -21.0), turned to 180 degrees
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Connections:
- J6 pad 1: +5V_MCU -> GND
- J6 pad 10: +3.3V_SENSORS -> /CH_D_MOSFET_ESP_MAIN_3V3
- J6 pad 11: +3.3V_SENSORS -> /CH_D_MOSFET_ESP_MAIN_3V3
- J6 pad 13: /RX_UART_BUS1_3V3 -> /CH_C_MOSFET_ESP_MAIN_3V3
- J6 pad 14: /RX_UART_BUS1_3V3 -> /CH_C_MOSFET_ESP_MAIN_3V3
- J6 pad 15: /RX_UART_BUS1_3V3 -> /CH_C_MOSFET_ESP_MAIN_3V3
- J6 pad 17: /TX_UART_BUS1_3V3 -> +3.3V_SENSORS
- J6 pad 18: /TX_UART_BUS1_3V3 -> +3.3V_SENSORS
- J6 pad 19: /TX_UART_BUS1_3V3 -> +3.3V_SENSORS
- J6 pad 20: GND -> +3.3V_SENSORS
- J6 pad 4: GND -> +5V_MCU
- J6 pad 5: Net-(J6-Pin_5) -> GND
- J6 pad 6: Net-(J6-Pin_5) -> GND
- J6 pad 7: Net-(J6-Pin_5) -> GND
- J6 pad 9: +3.3V_SENSORS -> /CH_D_MOSFET_ESP_MAIN_3V3
- R10 pad 1: /CH_C_MOSFET_ESP_3V3 -> /CH_C_MOSFET_ESP_MAIN_3V3
- R11 pad 1: /CH_D_MOSFET_ESP2_3V3 -> /CH_D_MOSFET_ESP_CTR_3V3
- R12 pad 1: /CH_C_MOSFET_ESP2_3V3 -> /CH_C_MOSFET_ESP_CTR_3V3
- R8 pad 1: /CH_A_MOSFET_ESP2_3V3 -> /CH_A_MOSFET_ESP_CTR_3V3
- R9 pad 1: /CH_D_MOSFET_ESP_3V3 -> /CH_D_MOSFET_ESP_MAIN_3V3
Routing:
- net Net-(BOOST2-OUT+): track 0.00 -> 51.5 mm
- net Net-(BOOST2-IN+): track 0.00 -> 30.7 mm
- net +3.3V_SENSORS: track 0.00 -> 25.1 mm
- net Net-(J3-Pin_1): track 0.00 -> 23.6 mm
- net Net-(BOOST1-IN+): track 0.00 -> 21.4 mm
- net +5V_MCU: track 0.00 -> 15.8 mm
- net Net-(J4-Pin_1): track 0.00 -> 13.4 mm
