File: ELS-ELH/ELH/PCB_B/PCB_B.kicad_pcb (KiCad board)
At the start: 2 copper layers, 95 x 95 mm, 22 parts, among them J1 Pressure Transducer Input, J2 Conn_01x04_Pin, J3 Conn_01x20_Pin, J4 Conn_01x20_Pin, U1 GY-87

Commit message: Update on schematics B
Parts:
- removed ADC1: ADS1115, ELH_Library:ADS1115
- added J10: Conn_01x07_Pin, Connector_PinHeader_2.54mm:PinHeader_1x07_P2.54mm_Vertical, F.Cu at (156.0, 29.8)
- added J11: UART BUS 2 3V3, Connector_PinHeader_2.54mm:PinHeader_1x02_P2.54mm_Vertical, F.Cu at (142.9, 30.4)
- added J12: UART BUS 2 3V3, Connector_PinHeader_2.54mm:PinHeader_1x02_P2.54mm_Vertical, F.Cu at (147.5, 30.4)
- added J13: Conn_01x06_Pin, Connector_PinHeader_2.54mm:PinHeader_1x06_P2.54mm_Vertical, F.Cu at (161.1, -7.08)
- added J3: Conn_01x20_Pin, Connector_PinHeader_2.54mm:PinHeader_1x20_P2.54mm_Vertical, F.Cu at (118.3, -6.45)
- added J5: UART BUS 2 3V3, Connector_PinHeader_2.54mm:PinHeader_1x02_P2.54mm_Vertical, F.Cu at (138.3, 30.4)
- added J6: Conn_01x08_Pin, Connector_PinHeader_2.54mm:PinHeader_1x08_P2.54mm_Vertical, F.Cu at (163.3, 16.2)
- added J7: I2C Bus Connector 3, Connector_PinHeader_2.54mm:PinHeader_1x04_P2.54mm_Vertical, F.Cu at (138.1, 36.9)
- added J8: I2C Bus Connector 2, Connector_PinHeader_2.54mm:PinHeader_1x04_P2.54mm_Vertical, F.Cu at (142.2, 36.9)
- added J9: I2C Bus Connector 1, Connector_PinHeader_2.54mm:PinHeader_1x04_P2.54mm_Vertical, F.Cu at (146.4, 36.9)
- added R13: 100, Resistor_THT:R_Axial_DIN0207_L6.3mm_D2.5mm_P7.62mm_Horizontal, F.Cu at (126.8, 32.8)
- Bornera7: value UART BUS 2 -> UART BUS 2 5V
- ESP1, R4, R5, R7: moved to F.Cu
- J1: value Pressure Transducer Input -> Conn_01x07_Pin; footprint ELH_Library:Bornera 3P -> Connector_PinHeader_2.54mm:PinHeader_1x07_P2.54mm_Vertical
- J2: value Conn_01x04_Pin -> GPS Connector
- moved J1 189.8 mm to (151.8, 29.8), turned to 0 degrees
- moved C13 187.0 mm to (145.6, 11.1)
- moved C2 185.1 mm to (151.7, 9.85), turned to 0 degrees
- moved Bornera7 183.4 mm to (150.3, 15.3), turned to 0 degrees
- moved D10 172.5 mm to (128.7, 38.2)
- moved R4 166.9 mm to (126.8, 16.6), turned to 0 degrees
- moved R5 164.7 mm to (126.8, 20.6), turned to 0 degrees
- moved R7 162.6 mm to (126.8, 24.7), turned to 0 degrees
- moved J2 159.6 mm to (160.4, 30.4)
- moved BZ1 150.6 mm to (139.0, 21.3)
- moved BME2 144.7 mm to (140.2, 66.3), turned to 0 degrees
- moved W25QXX1 143.6 mm to (144.3, -7.97)
- moved R12 139.6 mm to (126.8, 28.7)
- moved U1 135.4 mm to (126.0, -8.00)
- moved SD_Adapter1 134.8 mm to (113.3, 88.1)
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Connections:
- Adapter1 pad 1: +3.3V -> +3.3V_SENSORS
- Adapter1 pad 10: /LED3 -> Net-(Adapter1-P5)
- Adapter1 pad 11: /LED2 -> Net-(Adapter1-P6)
- Adapter1 pad 12: /LED1 -> Net-(Adapter1-P7)
- Adapter1 pad 13: unconnected-(Adapter1-INT-Pad13) -> Net-(Adapter1-INT)
- Adapter1 pad 3: /I2C1_SDA -> /SDA_I2C_BUS1_3V3
- Adapter1 pad 4: /I2C1_SCL -> /SCL_I2C_BUS1_3V3
- Adapter1 pad 5: unconnected-(Adapter1-P0-Pad5) -> /CS_SD_3V3
- Adapter1 pad 6: /MOS1_2 -> Net-(Adapter1-P1)
- Adapter1 pad 7: /MOS2_2 -> Net-(Adapter1-P2)
- Adapter1 pad 8: unconnected-(Adapter1-P3-Pad8) -> Net-(Adapter1-P3)
- Adapter1 pad 9: /BUZZER1 -> Net-(Adapter1-P4)
- Bornera7 pad 1: /UART2_TX_1 -> Net-(Bornera7-Pin_1)
- Bornera7 pad 2: /UART2_RX_1 -> Net-(Bornera7-Pin_2)
- C13 pad 1: +5VA -> +5V_MCU
- C2 pad 2: +5VA -> +5V_MCU
- Converter1 pad 11: +3.3V -> +3.3V_SENSORS
- Converter1 pad 12: /I2C1_SCL -> /TX_UART_BUS2_3V3
- Converter1 pad 13: /I2C1_SDA -> /RX_UART_BUS2_3V3
- Converter1 pad 14: /UART2_TX_2 -> Net-(Converter1-A3)
- Converter1 pad 15: /UART2_RX_2 -> Net-(Converter1-A4)
- Converter1 pad 16: unconnected-(Converter1-A5-Pad16) -> Net-(Converter1-A5)
- Converter1 pad 17: unconnected-(Converter1-A6-Pad17) -> Net-(Converter1-A6)
- Converter1 pad 18: unconnected-(Converter1-A7-Pad18) -> Net-(Converter1-A7)
- Converter1 pad 19: unconnected-(Converter1-A8-Pad19) -> Net-(Converter1-A8)
- Converter1 pad 2: /I2C1_SCL_1 -> /TX_UART_BUS2_5V
- Converter1 pad 20: +3.3V -> Net-(Converter1-OE)
- Converter1 pad 3: /I2C1_SDA_1 -> /RX_UART_BUS2_5V
- Converter1 pad 4: /UART2_TX_1 -> Net-(Converter1-B3)
- Converter1 pad 5: /UART2_RX_1 -> Net-(Converter1-B4)
- Converter1 pad 6: unconnected-(Converter1-B5-Pad6) -> Net-(Converter1-B5)
- Converter1 pad 7: unconnected-(Converter1-B6-Pad7) -> Net-(Converter1-B6)
- Converter1 pad 8: unconnected-(Converter1-B7-Pad8) -> Net-(Converter1-B7)
- Converter1 pad 9: unconnected-(Converter1-B8-Pad9) -> Net-(Converter1-B8)
- J1 pad 1: /PT_ADC1 -> Net-(Converter1-OE)
- J1 pad 2: GND -> Net-(Converter1-A8)
- J1 pad 3: +5V -> Net-(Converter1-A7)
- J2 pad 2: /UART3_TX -> /TX_UART_BUS3_3V3
- J2 pad 3: /UART3_RX -> /RX_UART_BUS3_3V3
- J2 pad 4: +3.3V -> +3.3V_SENSORS
- J4 pad 1: unconnected-(J4-Pin_1-Pad1) -> +5V
- J4 pad 10: /MOS1_2 -> +3.3V_SENSORS
- J4 pad 11: +3.3V -> +3.3V_SENSORS
- J4 pad 12: +3.3V -> GND
- J4 pad 13: +3.3V -> /CH_D_MOSFET_ESP_3V3
- J4 pad 14: +5VA -> /CH_D_MOSFET_ESP_3V3
- J4 pad 15: +5VA -> /CH_D_MOSFET_ESP_3V3
- J4 pad 16: +5VA -> GND
- J4 pad 17: GND -> /CH_C_MOSFET_ESP_3V3
- J4 pad 18: /MOS2_2 -> /CH_C_MOSFET_ESP_3V3
- J4 pad 19: /MOS2_2 -> /CH_C_MOSFET_ESP_3V3
- J4 pad 2: GND -> +5V
- J4 pad 20: /MOS2_2 -> GND
- J4 pad 3: GND -> +5V
- J4 pad 5: +5V -> +5V_MCU
- J4 pad 6: +5V -> +5V_MCU
- J4 pad 7: +5V -> +5V_MCU
- J4 pad 8: /MOS1_2 -> GND
- J4 pad 9: /MOS1_2 -> +3.3V_SENSORS
- R12 pad 1: /BUZZER1 -> /BUZZER_SIGNAL_3V3
- R4 pad 2: /LED1 -> /LED_RED_SIGNAL_3V3
- R5 pad 2: /LED2 -> /LED_GREEN_SIGNAL_3V3
- R7 pad 2: /LED3 -> /LED_BLUE_SIGNAL_3V3
- SD_Adapter1 pad 1: +3.3V -> +3.3V_SENSORS
- SD_Adapter1 pad 2: /CS_SD -> /CS_SD_3V3
- SD_Adapter1 pad 3: /SPI2_MOSI -> /MOSI_SPI_BUS1_3V3
- SD_Adapter1 pad 4: /SPI2_SCK -> /SCK_SPI_BUS1_3V3
- SD_Adapter1 pad 5: /SPI2_MISO -> /MISO_SPI_BUS1_3V3
- U1 pad 2: +3.3V -> +3.3V_SENSORS
- U1 pad 4: /I2C1_SCL -> /SCL_I2C_BUS1_3V3
- U1 pad 5: /I2C1_SDA -> /SDA_I2C_BUS1_3V3
- W25QXX1 pad 1: +3.3V -> +3.3V_SENSORS
- W25QXX1 pad 2: /CS_FLASH -> /CS_FLASH_3V3
- W25QXX1 pad 3: /SPI1_MISO -> /MISO_SPI_BUS1_3V3
- W25QXX1 pad 5: /SPI1_SCK -> /SCK_SPI_BUS1_3V3
- W25QXX1 pad 6: /SPI1_MOSI -> /MOSI_SPI_BUS1_3V3
Routing:
- net +3.3V: track 238.3 -> 5.08 mm, vias 1 -> 0
- net +5VA: track 217.2 -> 5.08 mm, vias 1 -> 0
- net +5V: track 222.0 -> 31.5 mm
- net /SPI1_SCK: track 137.1 -> 0.00 mm
- net /SPI1_MOSI: track 130.3 -> 0.00 mm
- net /I2C1_SCL: track 128.0 -> 0.00 mm
- net /SPI1_MISO: track 123.5 -> 0.00 mm
- net /I2C1_SDA_1: track 119.3 -> 0.00 mm
- net /I2C1_SDA: track 113.0 -> 0.00 mm
- net /I2C1_SCL_1: track 110.2 -> 0.00 mm
- net /UART2_RX_1: track 108.4 -> 0.00 mm
- net /UART2_TX_1: track 94.4 -> 0.00 mm
- net /MOS1_2: track 85.3 -> 0.00 mm
- net /SPI2_MOSI: track 67.6 -> 0.00 mm
- net /SPI2_SCK: track 62.1 -> 0.00 mm
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Other:
- outline, holes or cut-outs redrawn
- board text removed: "D1"

Commit message: Update in PCB B - new layout
Parts:
- removed J1: Conn_01x07_Pin, Connector_PinHeader_2.54mm:PinHeader_1x07_P2.54mm_Vertical
- removed J11, J5: UART BUS 2 3V3, Connector_PinHeader_2.54mm:PinHeader_1x02_P2.54mm_Vertical
- removed the J3 at (-24.1, -44.0)
- added J14: TX2 3V3, Connector_PinSocket_2.54mm:PinSocket_1x01_P2.54mm_Vertical, F.Cu at (35.3, -27.2)
- added J15: RX2 3V3, Connector_PinSocket_2.54mm:PinSocket_1x01_P2.54mm_Vertical, F.Cu at (33.1, -19.8)
- added J16: TX2 5V, Connector_PinSocket_2.54mm:PinSocket_1x01_P2.54mm_Vertical, F.Cu at (32.0, -25.5)
- added J17: RX2 5V, Connector_PinSocket_2.54mm:PinSocket_1x01_P2.54mm_Vertical, F.Cu at (31.3, -23.0)
- added J18: Conn_01x06_Pin, Connector_PinHeader_2.54mm:PinHeader_1x06_P2.54mm_Vertical, F.Cu at (40.7, 11.4)
- added R14: 220, Resistor_THT:R_Axial_DIN0207_L6.3mm_D2.5mm_P7.62mm_Horizontal, F.Cu at (30.9, 15.7)
- ESP1: moved to B.Cu
- moved W25QXX1 187.7 mm to (-42.4, -27.3)
- moved J9 184.7 mm to (-37.9, 24.6), turned to 165 degrees
- moved J8 183.3 mm to (-40.6, 23.9), turned to 165 degrees
- moved J2 181.9 mm to (-18.2, -3.89)
- moved J7 181.8 mm to (-43.2, 23.2), turned to 165 degrees
- moved BZ1 172.0 mm to (-24.5, -32.1)
- moved J10 163.2 mm to (7.81, -38.6), turned to -90 degrees
- moved R13 158.7 mm to (-24.0, -16.7), turned to 90 degrees
- moved U1 158.5 mm to (-30.4, 17.6)
- moved SD_Adapter1 158.1 mm to (-23.4, 8.59), turned to 180 degrees
- moved Converter1 155.1 mm to (16.9, -8.02)
- moved BME2 152.4 mm to (12.8, -17.2), turned to 180 degrees
- moved R12 150.3 mm to (-16.4, -16.6), turned to 90 degrees
- moved J6 148.8 mm to (16.1, 38.5), turned to -90 degrees
- moved IMU3 147.4 mm to (-12.8, -10.2)
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Connections:
- BME2 pad 3Vo: (no net) -> +3.3V_SENSORS
- BME2 pad CS: (no net) -> /CS_BME_3V3
- BME2 pad GND: (no net) -> GND
- BME2 pad SCK: (no net) -> Net-(BME2-SCK)
- BME2 pad SD0: (no net) -> /MISO_SPI_BUS1_3V3
- BME2 pad SDI: (no net) -> /MOSI_SPI_BUS1_3V3
- BME2 pad VIN: (no net) -> unconnected-(BME2-PadVIN)
- Converter1 pad 1: +5V -> +5V_MCU
- ESP1 pad 3V3: (no net) -> unconnected-(ESP1-Pad3V3)
- ESP1 pad D12: (no net) -> /D12_ESP_3V3
- ESP1 pad D13: (no net) -> /LED_RED_SIGNAL_3V3
- ESP1 pad D14: (no net) -> /LED_GREEN_SIGNAL_3V3
- ESP1 pad D15: (no net) -> /D15_ESP_3V3
- ESP1 pad D18: (no net) -> /SCK_SPI_BUS1_3V3
- ESP1 pad D19: (no net) -> /MISO_SPI_BUS1_3V3
- ESP1 pad D2: (no net) -> /D2_ESP_3V3
- ESP1 pad D21: (no net) -> /SDA_I2C_BUS1_3V3
- ESP1 pad D22: (no net) -> /SCL_I2C_BUS1_3V3
- ESP1 pad D23: (no net) -> /MOSI_SPI_BUS1_3V3
- ESP1 pad D25: (no net) -> /TX_UART_BUS3_3V3
- ESP1 pad D26: (no net) -> /CS_BME_3V3
- ESP1 pad D27: (no net) -> /LED_BLUE_SIGNAL_3V3
- ESP1 pad D32: (no net) -> /TX_UART_BUS2_3V3
- ESP1 pad D33: (no net) -> /TX_UART_BUS1_3V3
- ESP1 pad D34: (no net) -> /RX_UART_BUS1_3V3
- ESP1 pad D35: (no net) -> /RX_UART_BUS2_3V3
- ESP1 pad D4: (no net) -> /CH_C_MOSFET_ESP_3V3
- ESP1 pad D5: (no net) -> /CS_FLASH_3V3
- ESP1 pad EN: (no net) -> /EN_ESP_3V3
- ESP1 pad GND: (no net) -> GND
- ESP1 pad RX0: (no net) -> /RX0_ESP_3V3
- ESP1 pad RX2: (no net) -> /CH_D_MOSFET_ESP_3V3
- ESP1 pad TX0: (no net) -> /TX0_ESP_3V3
- ESP1 pad TX2: (no net) -> /BUZZER_SIGNAL_3V3
- ESP1 pad VIN: (no net) -> +5V_MCU
- ESP1 pad VN: (no net) -> /D39_ESP_3V3
- ESP1 pad VP: (no net) -> /RX_UART_BUS3_3V3
- IMU3 pad 3V: (no net) -> +3.3V_SENSORS
- IMU3 pad ADR: (no net) -> unconnected-(IMU3-PadADR)
- IMU3 pad GND: (no net) -> GND
- IMU3 pad PS0: (no net) -> unconnected-(IMU3-PadPS0)
- IMU3 pad PS1: (no net) -> unconnected-(IMU3-PadPS1)
- IMU3 pad SCL: (no net) -> /SCL_I2C_BUS1_3V3
- IMU3 pad SDA: (no net) -> /SDA_I2C_BUS1_3V3
Routing:
- net +3.3V_SENSORS: track 0.00 -> 231.5 mm
- net /RX_UART_BUS2_3V3: track 0.00 -> 126.5 mm
- net /MISO_SPI_BUS1_3V3: track 0.00 -> 110.6 mm
- net /MOSI_SPI_BUS1_3V3: track 0.00 -> 99.5 mm
- net +5V_MCU: track 0.00 -> 97.7 mm
- net /TX_UART_BUS2_3V3: track 0.00 -> 88.4 mm
- net /SDA_I2C_BUS1_3V3: track 0.00 -> 85.5 mm
- net /SCL_I2C_BUS1_3V3: track 0.00 -> 80.0 mm
- net /CS_FLASH_3V3: track 0.00 -> 74.5 mm
- net /BUZZER_SIGNAL_3V3: track 0.00 -> 71.1 mm
- net /SCK_SPI_BUS1_3V3: track 0.00 -> 66.4 mm
- net /CH_D_MOSFET_ESP_3V3: track 0.00 -> 59.2 mm
- net /CH_C_MOSFET_ESP_3V3: track 0.00 -> 52.8 mm
- net /RX_UART_BUS1_3V3: track 0.00 -> 48.5 mm
- net /TX_UART_BUS1_3V3: track 0.00 -> 48.1 mm
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
Commit message: PCB B Almost finishhed
Parts:
- removed Adapter1: PCF8574, ELH_Library:PCF8574
- removed J12: UART BUS 2 3V3, Connector_PinHeader_2.54mm:PinHeader_1x02_P2.54mm_Vertical
- removed J6: Conn_01x08_Pin, Connector_PinHeader_2.54mm:PinHeader_1x08_P2.54mm_Vertical
- added BZ2: Buzzer, Buzzer_Beeper:Buzzer_12x9.5RM7.6, F.Cu at (40.0, -23.0)
- added C1: C_Small, Capacitor_THT:C_Disc_D5.0mm_W2.5mm_P5.00mm, F.Cu at (-27.6, -27.2)
- added C3: C_Small, Capacitor_THT:C_Disc_D5.0mm_W2.5mm_P5.00mm, F.Cu at (-32.6, -24.0)
- added C4: C_Small, Capacitor_THT:C_Disc_D5.0mm_W2.5mm_P5.00mm, F.Cu at (-15.0, -8.00)
- added C5: C_Polarized_Small, Capacitor_THT:CP_Radial_D5.0mm_P2.50mm, F.Cu at (-19.0, -3.00)
- added D1: LED_RKGB, LED_THT:LED_D5.0mm-4_RGB_Staggered_Pins, F.Cu at (-14.5, 6.25)
- added ESP2: ESP32 DEVKIT V1, ELH_Library:ESP32 DEVKIT V1, B.Cu at (0.00, -25.0)
- added J11: Conn_01x08_Pin, Connector_PinSocket_2.54mm:PinSocket_1x08_P2.54mm_Vertical, F.Cu at (-35.9, -32.2)
- added J19: ~, Connector_PinSocket_2.54mm:PinSocket_1x01_P2.54mm_Vertical, F.Cu at (-32.5, 2.20)
- added J20: ~, Connector_PinSocket_2.54mm:PinSocket_1x01_P2.54mm_Vertical, F.Cu at (-32.5, -2.00)
- added R1: R_US, Resistor_THT:R_Axial_DIN0207_L6.3mm_D2.5mm_P7.62mm_Horizontal, F.Cu at (-30.0, -30.0)
- added R2: R_US, Resistor_THT:R_Axial_DIN0207_L6.3mm_D2.5mm_P7.62mm_Horizontal, F.Cu at (-30.0, -20.5)
- added R3: R_US, Resistor_THT:R_Axial_DIN0207_L6.3mm_D2.5mm_P7.62mm_Horizontal, F.Cu at (28.4, -33.0)
- added R6: R_US, Resistor_THT:R_Axial_DIN0207_L6.3mm_D2.5mm_P7.62mm_Horizontal, B.Cu at (-2.50, 3.87)
- added R8: R_US, Resistor_THT:R_Axial_DIN0207_L6.3mm_D2.5mm_P7.62mm_Horizontal, B.Cu at (-6.00, 3.87)
- added R9: R_US, Resistor_THT:R_Axial_DIN0207_L6.3mm_D2.5mm_P7.62mm_Horizontal, B.Cu at (-9.50, 3.87)
- R4, R5, R7, SD_Adapter1: moved to B.Cu
- moved W25QXX1 98.7 mm to (35.7, 33.0), turned to 180 degrees
- moved J3 88.0 mm to (-24.1, 44.0)
- moved J4 88.0 mm to (-24.1, -44.0)
- moved J9 81.6 mm to (41.0, 3.80), turned to 180 degrees
- moved J8 80.1 mm to (37.0, 3.80), turned to 180 degrees
- moved J7 78.7 mm to (33.0, 3.80), turned to 180 degrees
- moved Bornera7 71.8 mm to (-35.4, -5.05), turned to -90 degrees
- moved J16 71.7 mm to (-32.5, 5.89), turned to 0 degrees
- moved J14 70.6 mm to (-28.9, 2.20), turned to 0 degrees
- moved R13 69.9 mm to (39.1, 13.5), turned to 180 degrees
- moved J10 67.3 mm to (68.1, -8.71), turned to 180 degrees
- moved J17 66.1 mm to (-32.5, -5.75), turned to 0 degrees
- moved J15 64.5 mm to (-28.9, -2.00), turned to 0 degrees
- moved BZ1 57.3 mm to (-40.0, 23.0)
- moved R12 54.5 mm to (-28.8, 36.5), turned to 180 degrees
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Connections:
- net /BUZZER_SIGNAL_3V3 renamed /BUZZER_SIGNAL_ESP_MAIN_3V3
- net /CS_BME_3V3 renamed /CS_BME_ESP_MAIN_3V3
- net /CS_FLASH_3V3 renamed /CS_FLASH_ESP_MAIN_3V3
- net /LED_BLUE_SIGNAL_3V3 renamed /LED_BLUE_SIGNAL_ESP_MAIN_3V3
- net /LED_GREEN_SIGNAL_3V3 renamed /LED_GREEN_SIGNAL_ESP_MAIN_3V3
- net /LED_RED_SIGNAL_3V3 renamed /LED_RED_SIGNAL_ESP_MAIN_3V3
- net /MISO_SPI_BUS1_3V3 renamed /MISO_SPI_BUS1_ESP_MAIN_3V3
- net /MOSI_SPI_BUS1_3V3 renamed /MOSI_SPI_BUS1_ESP_MAIN_3V3
- net /RX_UART_BUS2_3V3 renamed /RX_UART_BUS2_ESP_MAIN_3V3
- net /RX_UART_BUS3_3V3 renamed /RX_UART_BUS3_ESP_MAIN_3V3
- net /SCK_SPI_BUS1_3V3 renamed /SCK_SPI_BUS1_ESP_MAIN_3V3
- net /SCL_I2C_BUS1_3V3 renamed /SCL_I2C_BUS1_ESP_MAIN_3V3
- net /SDA_I2C_BUS1_3V3 renamed /SDA_I2C_BUS1_ESP_MAIN_3V3
- net /TX_UART_BUS2_3V3 renamed /TX_UART_BUS2_ESP_MAIN_3V3
- net /TX_UART_BUS3_3V3 renamed /TX_UART_BUS3_ESP_MAIN_3V3
- ESP1 pad D12: /D12_ESP_3V3 -> /D12_ESP_ESP_MAIN_3V3
- ESP1 pad D15: /D15_ESP_3V3 -> /D15_ESP_MAIN_3V3
- ESP1 pad D2: /D2_ESP_3V3 -> /D2_ESP_MAIN_3V3
- ESP1 pad D33: /TX_UART_BUS1_3V3 -> /TX_UART_BUS1_ESP_MAIN_3V3
- ESP1 pad D34: /RX_UART_BUS1_3V3 -> /RX_UART_BUS1_ESP_MAIN_3V3
- ESP1 pad D4: /CH_C_MOSFET_ESP_3V3 -> /CH_C_MOSFET_ESP_MAIN_3V3
- ESP1 pad EN: /EN_ESP_3V3 -> /EN_ESP_MAIN_3V3
- ESP1 pad RX0: /RX0_ESP_3V3 -> /RX0_ESP_MAIN_3V3
- ESP1 pad RX2: /CH_D_MOSFET_ESP_3V3 -> /CH_D_MOSFET_ESP_MAIN_3V3
- ESP1 pad TX0: /TX0_ESP_3V3 -> /TX0_ESP_ESP_MAIN_3V3
- ESP1 pad VN: /D39_ESP_3V3 -> /D39_ESP_ESP_MAIN_3V3
- J13 pad 1: Net-(Converter1-B3) -> Net-(Converter1-B8)
- J13 pad 2: Net-(Converter1-B4) -> Net-(Converter1-B7)
- J13 pad 3: Net-(Converter1-B5) -> Net-(Converter1-B6)
- J13 pad 4: Net-(Converter1-B6) -> Net-(Converter1-B5)
- J13 pad 5: Net-(Converter1-B7) -> Net-(Converter1-B4)
- J13 pad 6: Net-(Converter1-B8) -> Net-(Converter1-B3)
- J3 pad 1: +5V_MCU -> GND
- J3 pad 10: +3.3V_SENSORS -> /CH_D_MOSFET_ESP_MAIN_3V3
- J3 pad 11: +3.3V_SENSORS -> /CH_D_MOSFET_ESP_MAIN_3V3
- J3 pad 13: /RX_UART_BUS1_3V3 -> /CH_C_MOSFET_ESP_MAIN_3V3
- J3 pad 14: /RX_UART_BUS1_3V3 -> /CH_C_MOSFET_ESP_MAIN_3V3
- J3 pad 15: /RX_UART_BUS1_3V3 -> /CH_C_MOSFET_ESP_MAIN_3V3
- J3 pad 17: /TX_UART_BUS1_3V3 -> +3.3V_SENSORS
- J3 pad 18: /TX_UART_BUS1_3V3 -> +3.3V_SENSORS
- J3 pad 19: /TX_UART_BUS1_3V3 -> +3.3V_SENSORS
- J3 pad 20: GND -> +3.3V_SENSORS
- J3 pad 4: GND -> +5V_MCU
- J3 pad 5: +5V -> GND
- J3 pad 6: +5V -> GND
- J3 pad 7: +5V -> GND
- J3 pad 9: +3.3V_SENSORS -> /CH_D_MOSFET_ESP_MAIN_3V3
- J4 pad 1: +5V -> +3.3V_SENSORS
- J4 pad 10: +3.3V_SENSORS -> GND
- J4 pad 11: +3.3V_SENSORS -> /CH_D_MOSFET_ESP_CTR_3V3
- J4 pad 12: GND -> /CH_D_MOSFET_ESP_CTR_3V3
- J4 pad 13: /CH_D_MOSFET_ESP_3V3 -> /CH_D_MOSFET_ESP_CTR_3V3
- J4 pad 14: /CH_D_MOSFET_ESP_3V3 -> GND
- J4 pad 15: /CH_D_MOSFET_ESP_3V3 -> /CH_C_MOSFET_ESP_CTR_3V3
- J4 pad 16: GND -> /CH_C_MOSFET_ESP_CTR_3V3
- J4 pad 17: /CH_C_MOSFET_ESP_3V3 -> /CH_C_MOSFET_ESP_CTR_3V3
- J4 pad 18: /CH_C_MOSFET_ESP_3V3 -> GND
- J4 pad 19: /CH_C_MOSFET_ESP_3V3 -> +3.3V_SENSORS
- J4 pad 2: +5V -> GND
- J4 pad 20: GND -> +3.3V_SENSORS
- J4 pad 3: +5V -> /CH_B_MOSFET_ESP_CTR_3V3
- J4 pad 4: GND -> /CH_B_MOSFET_ESP_CTR_3V3
- J4 pad 5: +5V_MCU -> /CH_B_MOSFET_ESP_CTR_3V3
- J4 pad 6: +5V_MCU -> GND
- J4 pad 7: +5V_MCU -> /CH_A_MOSFET_ESP_CTR_3V3
- J4 pad 8: GND -> /CH_A_MOSFET_ESP_CTR_3V3
- J4 pad 9: +3.3V_SENSORS -> /CH_A_MOSFET_ESP_CTR_3V3
- SD_Adapter1 pad 2: /CS_SD_3V3 -> /CS_SD_ESP_MAIN_3V3
Routing:
- net +3.3V_SENSORS: track 231.5 -> 487.2 mm, vias 0 -> 1
- net /TX_UART_BUS1_ESP_MAIN_3V3: track 0.00 -> 123.6 mm
- net +5V_MCU: track 97.7 -> 195.8 mm
- net /RX_UART_BUS1_ESP_MAIN_3V3: track 0.00 -> 95.4 mm
- net /TX_UART_BUS2_5V: track 26.1 -> 92.7 mm
- net Net-(ESP2-PadD34): track 0.00 -> 63.4 mm
- net /CH_D_MOSFET_ESP_3V3: track 59.2 -> 0.00 mm
- net /RPWM_BTS7960_ESP_CTR_3V3: track 0.00 -> 59.1 mm
- net /RX_UART_BUS2_5V: track 19.6 -> 74.3 mm
- net /CH_C_MOSFET_ESP_3V3: track 52.8 -> 0.00 mm
- net /RX_UART_BUS1_3V3: track 48.5 -> 0.00 mm
- net /TX_UART_BUS1_3V3: track 48.1 -> 0.00 mm
- net /TX_UART_BUS2_ESP_MAIN_3V3: track 88.4 -> 134.3 mm, vias 0 -> 1
- net /LPWM_BTS7960_ESP_CTR_3V3: track 0.00 -> 41.8 mm
- net Net-(ESP2-PadD35): track 0.00 -> 38.7 mm
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Other:
- outline, holes or cut-outs redrawn
