File: ELS-ELH/ELH/PCB_B/PCB_B.kicad_sch (KiCad schematic)
At the start: 22 parts, among them J1 Pressure Transducer Input, J2 GPS Connector, J3 Conn_01x20_Pin, J4 Conn_01x20_Pin, U1 GY-87

Commit message: Update on schematics B
Parts:
- removed ADC1: ADS1115, ELH_Library:ADS1115, symbol ELH_Library:ADS1115
- removed J1: Pressure Transducer Input, ELH_Library:Bornera 3P, symbol Connector:Screw_Terminal_01x03
- added J10: Conn_01x07_Pin, Connector_PinHeader_1.27mm:PinHeader_1x07_P1.27mm_Vertical, symbol Connector:Conn_01x07_Pin
- added J11, J12, J5: UART BUS 2 3V3, Connector_PinHeader_2.54mm:PinHeader_1x02_P2.54mm_Vertical, symbol Connector:Conn_01x02_Pin
- added J6: Conn_01x08_Pin, Connector_PinHeader_1.27mm:PinHeader_1x08_P1.27mm_Vertical, symbol Connector:Conn_01x08_Pin
- added J7: I2C Bus Connector 3, Connector_PinHeader_1.27mm:PinHeader_1x04_P1.27mm_Vertical, symbol Connector:Conn_01x04_Pin
- added J8: I2C Bus Connector 2, Connector_PinHeader_1.27mm:PinHeader_1x04_P1.27mm_Vertical, symbol Connector:Conn_01x04_Pin
- added J9: I2C Bus Connector 1, Connector_PinHeader_1.27mm:PinHeader_1x04_P1.27mm_Vertical, symbol Connector:Conn_01x04_Pin
- added R13: 100, Resistor_THT:R_Axial_DIN0207_L6.3mm_D2.5mm_P7.62mm_Horizontal, symbol Device:R_US
Connections:
- net +3.3V_SENSORS: now also J7.4 (Pin_4), J8.4 (Pin_4), J9.4 (Pin_4)
- net BUZZER_SIGNAL_3V3: now also ESP1.22 (D17); no longer Adapter1.9 (P4)
- net CH_C_MOSFET_ESP_3V3: now also ESP1.20 (D4); no longer Adapter1.6 (P1)
- net CH_D_MOSFET_ESP_3V3: now also ESP1.21 (D16); no longer Adapter1.7 (P2)
- net CS_SD_3V3: now also Adapter1.5 (P0); no longer ESP1.13 (D13)
- net GND: now also J7.3 (Pin_3), J8.3 (Pin_3), J9.3 (Pin_3)
- net LED_BLUE_SIGNAL_3V3: now also ESP1.10 (D27); no longer Adapter1.10 (P5)
- net LED_GREEN_SIGNAL_3V3: now also ESP1.11 (D14); no longer Adapter1.11 (P6)
- net LED_RED_SIGNAL_3V3: now also ESP1.13 (D13); no longer Adapter1.12 (P7)
- net MISO_SPI_BUS1_3V3: now also SD_Adapter1.5 (MISO)
- net MOSI_SPI_BUS1_3V3: now also SD_Adapter1.3 (MOSI)
- net RX_UART_BUS2_3V3: now also J5.2 (Pin_2)
- net RX_UART_BUS2_5V: now also J11.2 (Pin_2); no longer Bornera7.1 (Pin_1)
- net SCK_SPI_BUS1_3V3: now also SD_Adapter1.4 (CLK), R13.1; no longer BME2.4 (SCK)
- net SCL_I2C_BUS1_3V3: now also J7.2 (Pin_2), J8.2 (Pin_2), J9.2 (Pin_2)
- net SDA_I2C_BUS1_3V3: now also J7.1 (Pin_1), J8.1 (Pin_1), J9.1 (Pin_1)
- net TX_UART_BUS1_3V3: now also ESP1.7 (D33); no longer ESP1.8 (D25)
- net TX_UART_BUS2_3V3: now also ESP1.6 (D32), J5.1 (Pin_1); no longer ESP1.7 (D33)
- net TX_UART_BUS2_5V: now also J11.1 (Pin_1); no longer Bornera7.2 (Pin_2)
- net TX_UART_BUS3_3V3: now also ESP1.8 (D25); no longer ESP1.6 (D32)
- net EN_ESP_3V3: now reaches ESP1.1 (EN)
- net EN_ESP_3V3: now also J10.7 (Pin_7)
- net D12_ESP_3V3: now reaches ESP1.12 (D12)
- net D12_ESP_3V3: now also J10.5 (Pin_5)
- net D15_ESP_3V3: now reaches ESP1.18 (D15)
- net D15_ESP_3V3: now also J10.1 (Pin_1)
- net D2_ESP_3V3: now reaches ESP1.19 (D2)
- net D2_ESP_3V3: now also J10.2 (Pin_2)
- net RX0_ESP_3V3: now reaches ESP1.27 (RX0)
- net RX0_ESP_3V3: now also J10.3 (Pin_3)
- net TX0_ESP_3V3: now reaches ESP1.28 (TX0)
- net TX0_ESP_3V3: now also J10.4 (Pin_4)
- net D39_ESP_3V3: now reaches ESP1.3 (39/VN)
- net D39_ESP_3V3: now also J10.6 (Pin_6)
- net at Adapter1.13 (INT): now also J6.1 (Pin_1)
- net at Adapter1.8 (P3): now also J6.6 (Pin_6)
- removed net MISO_SPI_BUS2_3V3: ESP1.10 (D27), SD_Adapter1.5 (MISO)
- removed net MOSI_SPI_BUS2_3V3: ESP1.22 (D17), SD_Adapter1.3 (MOSI)
- removed net SCK_SPI_BUS2_3V3: ESP1.21 (D16), SD_Adapter1.4 (CLK)
- new net: Adapter1.10 (P5), J6.4 (Pin_4)
- new net: Adapter1.11 (P6), J6.3 (Pin_3)
- new net: Adapter1.12 (P7), J6.2 (Pin_2)
- new net: Adapter1.6 (P1), J6.8 (Pin_8)
- new net: Adapter1.7 (P2), J6.7 (Pin_7)
- new net: Adapter1.9 (P4), J6.5 (Pin_5)
- new net: Bornera7.1 (Pin_1), J12.1 (Pin_1)
- new net: Bornera7.2 (Pin_2), J12.2 (Pin_2)
- new net: BME2.4 (SCK), R13.2
- no-connect marks 36 -> 19
Other:
- note removed: "Headers"
- note removed: "LEDs MAIN OBC"
- note removed: "MAIN OBC (ESP32 WROOM 32)"
- note removed: "PCF8574"
- moved on the sheet: J2, J3, J4

Commit message: Update in PCB B - new layout
Parts:
- removed J11, J5: UART BUS 2 3V3, Connector_PinHeader_2.54mm:PinHeader_1x02_P2.54mm_Vertical, symbol Connector:Conn_01x02_Pin
- added J13, J18: Conn_01x06_Pin, Connector_PinHeader_2.54mm:PinHeader_1x06_P2.54mm_Vertical, symbol Connector:Conn_01x06_Pin
- added J14: TX2 3V3, Connector_PinSocket_2.54mm:PinSocket_1x01_P2.54mm_Vertical, symbol Connector:Conn_01x01_Pin
- added J15: RX2 3V3, Connector_PinSocket_2.54mm:PinSocket_1x01_P2.54mm_Vertical, symbol Connector:Conn_01x01_Pin
- added J16: TX2 5V, Connector_PinSocket_2.54mm:PinSocket_1x01_P2.54mm_Vertical, symbol Connector:Conn_01x01_Pin
- added J17: RX2 5V, Connector_PinSocket_2.54mm:PinSocket_1x01_P2.54mm_Vertical, symbol Connector:Conn_01x01_Pin
- added R14: 220, Resistor_THT:R_Axial_DIN0207_L6.3mm_D2.5mm_P7.62mm_Horizontal, symbol Device:R_US
- J10: footprint Connector_PinHeader_1.27mm:PinHeader_1x07_P1.27mm_Vertical -> Connector_PinHeader_2.54mm:PinHeader_1x07_P2.54mm_Vertical
- J6: footprint Connector_PinHeader_1.27mm:PinHeader_1x08_P1.27mm_Vertical -> Connector_PinHeader_2.54mm:PinHeader_1x08_P2.54mm_Vertical
- J7, J8, J9: footprint Connector_PinHeader_1.27mm:PinHeader_1x04_P1.27mm_Vertical -> Connector_PinHeader_2.54mm:PinHeader_1x04_P2.54mm_Vertical
Connections:
- net SCL_I2C_BUS1_5V is gone; now on net TX_UART_BUS2_5V: Converter1.2 (B1)
- net SDA_I2C_BUS1_5V is gone; now on net RX_UART_BUS2_5V: Converter1.3 (B2)
- net +3.3V_SENSORS: now also BME2.3Vo (3V0), IMU3.3V, R14.1; no longer BME2.2 (3VO), IMU3.2 (3V)
- net +5V: no longer Converter1.1 (VB)
- net +5V_MCU: now also Converter1.1 (VB), ESP1.VIN; no longer ESP1.15 (VIN)
- net BUZZER_SIGNAL_3V3: now also ESP1.TX2 (D17/TX2); no longer ESP1.22 (D17)
- net CH_C_MOSFET_ESP_3V3: now also ESP1.D4; no longer ESP1.20 (D4)
- net CH_D_MOSFET_ESP_3V3: now also ESP1.RX2 (D16/RX2); no longer ESP1.21 (D16)
- net CS_BME_3V3: now also BME2.CS, ESP1.D26; no longer BME2.7 (CS), ESP1.23 (D5)
- net CS_FLASH_3V3: now also ESP1.D5; no longer ESP1.9 (D26)
- net D12_ESP_3V3: now also ESP1.D12; no longer ESP1.12 (D12)
- net D15_ESP_3V3: now also ESP1.D15; no longer ESP1.18 (D15)
- net D2_ESP_3V3: now also ESP1.D2; no longer ESP1.19 (D2)
- net D39_ESP_3V3: now also ESP1.VN (39/VN); no longer ESP1.3 (39/VN)
- net EN_ESP_3V3: now also ESP1.EN; no longer ESP1.1 (EN)
- net GND: now also BME2.GND, ESP1.GND, IMU3.GND; no longer BME2.3 (GND), ESP1.14 (GND), ESP1.17 (GND), IMU3.3 (GND)
- net LED_BLUE_SIGNAL_3V3: now also ESP1.D27; no longer ESP1.10 (D27)
- net LED_GREEN_SIGNAL_3V3: now also ESP1.D14; no longer ESP1.11 (D14)
- net LED_RED_SIGNAL_3V3: now also ESP1.D13; no longer ESP1.13 (D13)
- net MISO_SPI_BUS1_3V3: now also BME2.SD0, ESP1.D19; no longer BME2.5 (SDO), ESP1.25 (D19)
- net MOSI_SPI_BUS1_3V3: now also BME2.SDI, ESP1.D23; no longer BME2.6 (SDI), ESP1.30 (D23)
- net RX0_ESP_3V3: now also ESP1.RX0; no longer ESP1.27 (RX0)
- net RX_UART_BUS1_3V3: now also ESP1.D34; no longer ESP1.4 (D34)
- net RX_UART_BUS2_3V3: now also Converter1.13 (A2), ESP1.D35, J15.1 (Pin_1); no longer Converter1.15 (A4), ESP1.5 (D35)
- net RX_UART_BUS2_5V: now also J17.1 (Pin_1); no longer Converter1.5 (B4)
- net RX_UART_BUS3_3V3: now also ESP1.VP (36/VP); no longer ESP1.2 (36/VP)
- net SCK_SPI_BUS1_3V3: now also ESP1.D18; no longer ESP1.24 (D18)
- net SCL_I2C_BUS1_3V3: now also ESP1.D22, IMU3.SCL (SCL/RX); no longer Converter1.12 (A1), ESP1.29 (D22), IMU3.4 (SCL/RX)
- net SDA_I2C_BUS1_3V3: now also ESP1.D21, IMU3.SDA (SDA/TX); no longer Converter1.13 (A2), ESP1.26 (D21), IMU3.5 (SDA/TX)
- net TX0_ESP_3V3: now also ESP1.TX0; no longer ESP1.28 (TX0)
- net TX_UART_BUS1_3V3: now also ESP1.D33; no longer ESP1.7 (D33)
- net TX_UART_BUS2_3V3: now also Converter1.12 (A1), ESP1.D32, J14.1 (Pin_1); no longer Converter1.14 (A3), ESP1.6 (D32)
- net TX_UART_BUS2_5V: now also J16.1 (Pin_1); no longer Converter1.4 (B3)
- net TX_UART_BUS3_3V3: now also ESP1.D25; no longer ESP1.8 (D25)
- net at Converter1.16 (A5): now also J18.4 (Pin_4)
- net at Converter1.17 (A6): now also J18.3 (Pin_3)
- net at Converter1.18 (A7): now also J18.2 (Pin_2)
- net at Converter1.19 (A8): now also J18.1 (Pin_1)
- net at Converter1.20 (OE): now also R14.2
- net at Converter1.6 (B5): now also J13.3 (Pin_3)
- net at Converter1.7 (B6): now also J13.4 (Pin_4)
- net at Converter1.8 (B7): now also J13.5 (Pin_5)
- net at Converter1.9 (B8): now also J13.6 (Pin_6)
- net at R13.2: now also BME2.SCK; no longer BME2.4 (SCK)
- new net: Converter1.14 (A3), J18.6 (Pin_6)
- new net: Converter1.15 (A4), J18.5 (Pin_5)
- new net: Converter1.4 (B3), J13.1 (Pin_1)
- new net: Converter1.5 (B4), J13.2 (Pin_2)
- no-connect marks 19 -> 10
Other:
- moved on the sheet: J2

Commit message: PCB B Almost finishhed
Parts:
- removed Adapter1: PCF8574, ELH_Library:PCF8574, symbol ELH_Library:PCF8574
- removed J12: UART BUS 2 3V3, Connector_PinHeader_2.54mm:PinHeader_1x02_P2.54mm_Vertical, symbol Connector:Conn_01x02_Pin
- removed J6: Conn_01x08_Pin, Connector_PinHeader_2.54mm:PinHeader_1x08_P2.54mm_Vertical, symbol Connector:Conn_01x08_Pin
- added BZ2: Buzzer, Buzzer_Beeper:Buzzer_12x9.5RM7.6, symbol Device:Buzzer
- added C1, C3, C4: C_Small, Capacitor_THT:C_Disc_D5.0mm_W2.5mm_P5.00mm, symbol Device:C_Small
- added C5: C_Polarized_Small, Capacitor_THT:CP_Radial_D5.0mm_P2.50mm, symbol Device:C_Polarized_Small
- added D1: LED_RKGB, LED_THT:LED_D5.0mm-4_RGB_Staggered_Pins, symbol Device:LED_RKGB
- added ESP2: ESP32 DEVKIT V1, ELH_Library:ESP32 DEVKIT V1, symbol ELH_Library:ESP32 DEVKIT V1
- added J11: Conn_01x08_Pin, Connector_PinSocket_2.54mm:PinSocket_1x08_P2.54mm_Vertical, symbol Connector:Conn_01x08_Pin
- added J19, J20: (no value), Connector_PinSocket_2.54mm:PinSocket_1x01_P2.54mm_Vertical, symbol Connector:Conn_01x01_Pin
- added R1, R2, R3, R6, R8, R9: R_US, Resistor_THT:R_Axial_DIN0207_L6.3mm_D2.5mm_P7.62mm_Horizontal, symbol Device:R_US
Connections:
- net +3.3V_SENSORS: now also J3.17 (Pin_17), J3.18 (Pin_18), J3.19 (Pin_19), J3.20 (Pin_20), J4.1 (Pin_1), J4.19 (Pin_19), J4.20 (Pin_20), J11.1 (Pin_1); no longer J3.10 (Pin_10), J3.11 (Pin_11), J3.9 (Pin_9), J4.10 (Pin_10), J4.11 (Pin_11), J4.9 (Pin_9)
- net +5V_MCU: now also J3.4 (Pin_4), C4.2, C5.1, ESP2.VIN; no longer J3.1 (Pin_1), J4.5 (Pin_5), J4.6 (Pin_6), J4.7 (Pin_7)
- net D12_ESP_3V3: no longer ESP1.D12
- net D15_ESP_3V3: no longer ESP1.D15
- net D2_ESP_3V3: no longer ESP1.D2
- net D39_ESP_3V3: no longer ESP1.VN (39/VN)
- net EN_ESP_3V3: no longer ESP1.EN
- net GND: now also J3.1 (Pin_1), J3.5 (Pin_5), J3.6 (Pin_6), J3.7 (Pin_7), J4.10 (Pin_10), J4.14 (Pin_14), J4.18 (Pin_18), J4.2 (Pin_2), J4.6 (Pin_6), BZ2.2 (-), C1.1, C3.2, C4.1, C5.2, D1.2 (K), ESP2.GND, J11.2 (Pin_2); no longer J3.20 (Pin_20), J3.4 (Pin_4), J4.12 (Pin_12), J4.16 (Pin_16), J4.20 (Pin_20), J4.4 (Pin_4), J4.8 (Pin_8)
- net RX0_ESP_3V3: no longer ESP1.RX0
- net SCL_I2C_BUS1_3V3: now also ESP2.D22; no longer ESP1.D22, IMU3.SCL (SCL/RX), J7.2 (Pin_2), J8.2 (Pin_2), J9.2 (Pin_2), U1.4 (SCL)
- net TX0_ESP_3V3: no longer ESP1.TX0
- net at Converter1.4 (B3): now also J13.6 (Pin_6); no longer J13.1 (Pin_1)
- net at Converter1.5 (B4): now also J13.5 (Pin_5); no longer J13.2 (Pin_2)
- net at Converter1.6 (B5): now also J13.4 (Pin_4); no longer J13.3 (Pin_3)
- net at Converter1.7 (B6): now also J13.3 (Pin_3); no longer J13.4 (Pin_4)
- net at Converter1.8 (B7): now also J13.2 (Pin_2); no longer J13.5 (Pin_5)
- net at Converter1.9 (B8): now also J13.1 (Pin_1); no longer J13.6 (Pin_6)
- net at Bornera7.1 (Pin_1): now also J20.1 (Pin_1)
- net at Bornera7.2 (Pin_2): now also J19.1 (Pin_1)
- removed net +5V: J3.5 (Pin_5), J3.6 (Pin_6), J3.7 (Pin_7), J4.1 (Pin_1), J4.2 (Pin_2), J4.3 (Pin_3)
- net BUZZER_SIGNAL_3V3 renamed BUZZER_SIGNAL_ESP_MAIN_3V3
- removed net CH_C_MOSFET_ESP_3V3: ESP1.D4, J4.17 (Pin_17), J4.18 (Pin_18), J4.19 (Pin_19)
- removed net CH_D_MOSFET_ESP_3V3: ESP1.RX2 (D16/RX2), J4.13 (Pin_13), J4.14 (Pin_14), J4.15 (Pin_15)
- net CS_BME_3V3 renamed CS_BME_ESP_MAIN_3V3
- net CS_FLASH_3V3 renamed CS_FLASH_ESP_MAIN_3V3
- net CS_SD_3V3 renamed CS_SD_ESP_MAIN_3V3
- net LED_BLUE_SIGNAL_3V3 renamed LED_BLUE_SIGNAL_ESP_MAIN_3V3
- net LED_GREEN_SIGNAL_3V3 renamed LED_GREEN_SIGNAL_ESP_MAIN_3V3
- net LED_RED_SIGNAL_3V3 renamed LED_RED_SIGNAL_ESP_MAIN_3V3
- net MISO_SPI_BUS1_3V3 renamed MISO_SPI_BUS1_ESP_MAIN_3V3
- net MOSI_SPI_BUS1_3V3 renamed MOSI_SPI_BUS1_ESP_MAIN_3V3
- net RX_UART_BUS1_3V3 renamed CH_C_MOSFET_ESP_MAIN_3V3
- net CH_C_MOSFET_ESP_MAIN_3V3: now also ESP1.D4; no longer ESP1.D34
- net RX_UART_BUS2_3V3 renamed RX_UART_BUS2_ESP_MAIN_3V3
- net RX_UART_BUS3_3V3 renamed RX_UART_BUS3_ESP_MAIN_3V3
- net SCK_SPI_BUS1_3V3 renamed SCK_SPI_BUS1_ESP_MAIN_3V3
- net SDA_I2C_BUS1_3V3 renamed SDA_I2C_BUS1_ESP_MAIN_3V3
- removed net TX_UART_BUS1_3V3: ESP1.D33, J3.17 (Pin_17), J3.18 (Pin_18), J3.19 (Pin_19)
- net TX_UART_BUS2_3V3 renamed TX_UART_BUS2_ESP_MAIN_3V3
- net TX_UART_BUS3_3V3 renamed TX_UART_BUS3_ESP_MAIN_3V3
- new net: D1.1 (RA), R9.1
- new net: D1.3 (GA), R8.1
- new net: D1.4 (BA), R6.1
- new net: BZ2.1 (+), R3.2
- new net: ESP2.D34, R1.2
- new net: ESP2.D35, R2.2
- new net BUZZER_SIGNAL_ESP_CTR_3V3: ESP2.D4, R3.1
- new net CH_A_MOSFET_ESP_CTR_3V3: ESP2.TX2 (D17/TX2), J4.7 (Pin_7), J4.8 (Pin_8), J4.9 (Pin_9)
- new net CH_B_MOSFET_ESP_CTR_3V3: ESP2.RX2 (D16/RX2), J4.3 (Pin_3), J4.4 (Pin_4), J4.5 (Pin_5)
- new net CH_C_MOSFET_ESP_CTR_3V3: ESP2.D19, J4.15 (Pin_15), J4.16 (Pin_16), J4.17 (Pin_17)
- new net CH_D_MOSFET_ESP_CTR_3V3: ESP2.D18, J4.11 (Pin_11), J4.12 (Pin_12), J4.13 (Pin_13)
- new net CH_D_MOSFET_ESP_MAIN_3V3: ESP1.RX2 (D16/RX2), J3.10 (Pin_10), J3.11 (Pin_11), J3.9 (Pin_9)
- new net D12_ESP_ESP_MAIN_3V3: ESP1.D12
- new net D15_ESP_MAIN_3V3: ESP1.D15
- new net D2_ESP_MAIN_3V3: ESP1.D2
- new net D39_ESP_ESP_MAIN_3V3: ESP1.VN (39/VN)
- new net EN_ESP_MAIN_3V3: ESP1.EN
- new net LED_BLUE_SIGNAL_ESP_CTR_3V3: ESP2.D32, R6.2
- new net LED_GREEN_SIGNAL_ESP_CTR_3V3: ESP2.D33, R8.2
- new net LED_RED_SIGNAL_ESP_CTR_3V3: ESP2.D13, R9.2
- new net LPWM_BTS7960_ESP_CTR_3V3: ESP2.D26, J11.8 (Pin_8)
- new net L_EN_BTS7960_ESP_CTR_3V3: ESP2.D14, J11.6 (Pin_6)
- new net L_IS_BTS7960_ESP_CTR_3V3: C3.1, J11.4 (Pin_4), R2.1
- new net RPWM_BTS7960_ESP_CTR_3V3: ESP2.D25, J11.7 (Pin_7)
- new net RX0_ESP_MAIN_3V3: ESP1.RX0
- new net RX_UART_BUS1_ESP_MAIN_3V3: ESP1.D34, ESP2.D23
- new net R_EN_BTS7960_ESP_CTR_3V3: ESP2.D27, J11.5 (Pin_5)
- new net R_IS_BTS7960_ESP_CTR_3V3: C1.2, J11.3 (Pin_3), R1.1
- new net SCL_I2C_BUS1_ESP_MAIN_3V3: ESP1.D22, IMU3.SCL (SCL/RX), J7.2 (Pin_2), J8.2 (Pin_2), J9.2 (Pin_2), U1.4 (SCL)
- new net SDA_I2C_BUS1_ESP_CTR_3V3: ESP2.D21
- new net TX0_ESP_ESP_MAIN_3V3: ESP1.TX0
- new net TX_UART_BUS1_ESP_MAIN_3V3: ESP1.D33, ESP2.D5
- no-connect marks 10 -> 12
Other:
- moved on the sheet: J13, J14, J15, J16, J17, J2, J4, J7, J8, J9
